File: Electronics/Schematic/Maze solver.kicad_sch (KiCad schematic)
At the start: 2 parts

Commit message: Add files via upload
Parts:
- removed A1: Arduino_Nano_RP2040_Connect, Module:Arduino_Nano, symbol MCU_Module:Arduino_Nano_RP2040_Connect
- added U5: ATmega328P-P, Package_DIP:DIP-28_W7.62mm, symbol MCU_Microchip_ATmega:ATmega328P-P
Connections:
- net +5V: now also U5.20 (AVCC), U5.7 (VCC)
- net GND: now also U5.22 (GND), U5.8 (GND)
- net IR 5: no longer names the net of A2.25 (A6)
- net IR 6: no longer names the net of A2.26 (A7)
- new net Ultrasound 1 Echo: U5.5 (PD3)
- new net Ultrasound 1 Trig: U5.4 (PD2)
- new net Ultrasound 2 Echo: U5.6 (PD4)
- new net Ultrasound 3 Echo: U5.11 (PD5)
- new net Ultrasound 4 Echo: U5.12 (PD6)
