File: Electronics/Schematic/Maze Solver Finalisation.kicad_sch (KiCad schematic)
At the start: 82 parts, among them J1 Power Supply, M1 Motor_Servo, M2 Motor_Servo, M3 Motor_Servo, M4 Motor_Servo, U5 ATmega328P-P, U7 LM358, U8 LM358

Commit message: Uploaded verified schematic and PCB
Parts:
- removed +5V1 (x2), +5V2 (x2), +5V3 (x2), +5V4 (x2), GND1 (x2), GND2, GND3 (x3), GND4 (x2), IR1.1 (x2), IR1.2 (x2), IR2.1 (x2), IR2.2 (x2), IR3.1 (x2), IR3.2 (x2), IR4.1 (x2), IR4.2 (x2): Conn_01x01_Pin, Connector_PinHeader_1.00mm:PinHeader_1x01_P1.00mm_Vertical, symbol Connector:Conn_01x01_Pin
- removed J1: Power Supply, Connector_BarrelJack:BarrelJack_GCT_DCJ200-10-A_Horizontal, symbol Connector:Barrel_Jack_Switch_MountingPin
- removed Pot: R_Potentiometer, symbol Device:R_Potentiometer
- removed SW: SW_Push, symbol Switch:SW_Push
- added C1, C2: 22pF, Capacitor_THT:C_Disc_D4.7mm_W2.5mm_P5.00mm, symbol Device:C
- added IR1, IR2, IR3, IR4, IRA1, IRA2, IRA3, IRA4, LCD1: Conn_01x04_Pin, Connector_PinHeader_2.54mm:PinHeader_1x04_P2.54mm_Vertical, symbol Connector:Conn_01x04_Pin
- added J2: Power Supply, Connector_BarrelJack:BarrelJack_GCT_DCJ200-10-A_Horizontal, symbol Connector:Barrel_Jack_Switch
- added SW1: SW_SPST, Connector_PinHeader_2.54mm:PinHeader_1x02_P2.54mm_Vertical, symbol Switch:SW_SPST
- added U1: ~, Connector_PinHeader_2.54mm:PinHeader_1x05_P2.54mm_Vertical, symbol Device:Potentiometer_Switch
- added Y1: Crystal, Crystal:Crystal_HC49-4H_Vertical, symbol Device:Crystal
- R1, R10, R11, R12, R13, R2, R25, R26, R3, R4, R5, R6, R7, R8, R9: footprint Resistor_THT:R_Axial_DIN0207_L6.3mm_D2.5mm_P10.16mm_Horizontal -> Resistor_SMD:R_1206_3216Metric_Pad1.30x1.75mm_HandSolder
- RV1, RV2, RV3, RV4: footprint Potentiometer_THT:Potentiometer_Alpha_RD901F-40-00D_Single_Vertical_CircularHoles -> Potentiometer_THT:Potentiometer_ACP_CA9-H2,5_Horizontal
- US1, US2, US3, US4: footprint Connector_PinHeader_1.00mm:PinHeader_1x04_P1.00mm_Vertical -> Connector_PinHeader_2.54mm:PinHeader_1x04_P2.54mm_Vertical
- renumbered V+in to V+in2, V+out to V+out2, V-in to V-in2, V-out to V-out2
Connections:
- net GND: now also A3.29 (GND), A3.4 (GND), M1.3 (-), M2.3 (-), M3.3 (-), M4.3 (-), R12.2, R13.2, R25.2, R26.2, U7.4 (V-), U8.4 (V-), V-out1.1 (Pin_1), V-out2.1 (Pin_1), C1.2, C2.1, IR1.1 (Pin_1), IR2.1 (Pin_1), IR3.1 (Pin_1), IR4.1 (Pin_1), LCD1.1 (Pin_1), U1.3, U1.4
- net at D6.1 (K), D8.2 (A), RV3.1: now also IRA3.4 (Pin_4)
- net at RV3.2: now also IRA3.2 (Pin_2)
- net at R1.2, R10.2, RV3.3: now also IRA3.1 (Pin_1)
- net at D1.1 (K), D2.2 (A), RV1.1: now also IRA1.4 (Pin_4)
- net at RV1.2: now also IRA1.2 (Pin_2)
- net at R2.2, R3.2, RV1.3: now also IRA1.1 (Pin_1)
- net at V+in1.1 (Pin_1), V+in2.1 (Pin_1): now also SW1.2 (B)
- net at V-in1.1 (Pin_1), V-in2.1 (Pin_1): now also J2.2, J2.3
- net +5V: now reaches U5.20 (AVCC), U5.7 (VCC), US1.1 (Pin_1), US2.1 (Pin_1), US3.1 (Pin_1), US4.1 (Pin_1)
- net +5V: now also A3.30 (VIN), V+out2.1 (Pin_1)
- net at U5.10 (XTAL2/PB7): now also C2.2, Y1.1
- net at U5.9 (XTAL1/PB6): now also C1.1, Y1.2
- net at A3.27 (VUSB/5V), R7.2, R8.2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: now also IR1.4 (Pin_4), IR2.4 (Pin_4), IR3.4 (Pin_4), IR4.4 (Pin_4), LCD1.2 (Pin_2)
- net at D1.2 (A), R2.1: now also IRA1.3 (Pin_3)
- net at U8.6 (-): now also IR2.2 (Pin_2)
- net at D6.2 (A), R1.1: now also IRA3.3 (Pin_3)
- net at D3.2 (A), D4.1 (K), RV2.1: now also IRA2.4 (Pin_4)
- net at RV2.2: now also IRA2.2 (Pin_2)
- net at R4.2, R5.2, RV2.3: now also IRA2.1 (Pin_1)
- net at U8.5 (+): now also IR2.3 (Pin_3)
- net at R11.2, R6.2, RV4.3: now also IRA4.1 (Pin_1)
- net at D7.2 (A), R6.1: now also IRA4.3 (Pin_3)
- net at U7.2 (-): now also IR3.2 (Pin_2)
- net at D7.1 (K), D9.2 (A), RV4.1: now also IRA4.4 (Pin_4)
- net at RV4.2: now also IRA4.2 (Pin_2)
- net at D4.2 (A), R5.1: now also IRA2.3 (Pin_3)
- net at R8.1: now also A3.10 (D7), U1.2; no longer A3.9 (D6)
- net at U8.2 (-): now also IR1.2 (Pin_2)
- net at U8.3 (+): now also IR1.3 (Pin_3)
- net at U7.3 (+): now also IR3.3 (Pin_3)
- net at U7.6 (-): now also IR4.2 (Pin_2)
- net at A3.11 (D8), R7.1: now also U1.5
- net at R9.1: now also A3.9 (D6), U1.1; no longer A3.10 (D7)
- net at U7.5 (+): now also IR4.3 (Pin_3)
- net at A3.23 (SDA/A4): now also LCD1.3 (Pin_3)
- net at A3.24 (SCL/A5): now also LCD1.4 (Pin_4)
- new net: J2.1, SW1.1 (A)
Other:
- note added: "1"
- note added: "2"
- note added: "GND"
- note added: "SCL"
- note added: "SDA"
- note added: "Vcc"
- moved on the sheet: U5
