File: Electronics/PCB/Maze solver.kicad_pcb (KiCad board)
At the start: 2 copper layers, 153 x 86.5 mm, 29 parts, among them U1 LM358, U5 ATmega328P-P

Commit message: Updated PCB
Parts:
- removed the D3 at (228.7, 73.8)
- removed the D3 at (228.7, 40.3)
- removed the D3 at (84.8, 66.7)
- removed the D4 at (228.5, 67.0)
- removed the D4 at (85.0, 73.5)
- removed the D4 at (228.5, 33.5)
- removed the R5 at (226.6, 79.5)
- removed the R5 at (86.9, 61.0)
- removed the R5 at (226.6, 46.0)
- removed the R6 at (89.0, 74.1)
- removed the R6 at (224.5, 32.9)
- removed the R6 at (224.5, 66.4)
- removed the REF** at (99.5, 65.5)
- removed the REF** at (214.0, 75.0)
- removed the REF** at (214.0, 41.5)
- added REF**: Crystal_SMD_HC49-SD_HandSoldering, Crystal:Crystal_SMD_HC49-SD_HandSoldering, F.Cu at (154.1, 104.5)
- added REF**: C_Disc_D3.0mm_W1.6mm_P2.50mm, Capacitor_THT:C_Disc_D3.0mm_W1.6mm_P2.50mm, F.Cu at (157.8, 109.0)
- added REF**: C_Disc_D3.0mm_W1.6mm_P2.50mm, Capacitor_THT:C_Disc_D3.0mm_W1.6mm_P2.50mm, F.Cu at (146.2, 109.0)
Routing:
- net +5V: track 568.4 -> 311.5 mm, vias 20 -> 11
- net Ultrasound 1 Trig: track 0.00 -> 93.3 mm, vias 0 -> 4
- net (no net): track 140.8 -> 73.2 mm, vias 50 -> 31
- net Ultrasound 1 GND: track 90.6 -> 156.1 mm, vias 4 -> 5
- net Ultrasound 3 Echo: track 8.74 -> 59.1 mm
- net Ultrasound 2 Echo: track 7.45 -> 39.0 mm
- net Ultrasound 1 Vcc: track 74.7 -> 102.2 mm, vias 5 -> 4
- net unconnected-(U5-XTAL1/PB6-Pad9): track 0.00 -> 15.3 mm, vias 0 -> 1
- net unconnected-(U5-XTAL2/PB7-Pad10): track 0.00 -> 12.7 mm, vias 0 -> 1
- net Ultrasound 4 Echo: track 11.6 -> 15.0 mm, vias 1 -> 2
- net Ultrasound 1 Echo: track 14.7 -> 13.0 mm
Other:
- board size 153 x 86.5 mm -> 97.5 x 89 mm
